File: processor_attempt_1/processor_attempt_1.kicad_sch (KiCad schematic)
At the start: 337 parts, among them J1 Conn_01x03_Pin, J10 Conn_01x10_Pin, J11 Conn_01x10_Pin, J12 Conn_01x10_Pin, J13 Conn_01x10_Pin, J14 Conn_01x06_Pin, J15 Conn_01x06_Pin, J16 Conn_01x06_Pin, J17 Conn_01x06_Pin, J18 Conn_01x10_Pin, J19 Conn_01x10_Pin, J2 Conn_Coaxial, J20 Conn_01x08_Pin, J21 DB9_Female_MountingHoles, J22 Conn_01x08_Pin, J23 Conn_01x08_Pin, J24 Conn_01x08_Pin, J25 Conn_01x08_Pin, J26 Conn_01x08_Pin, J27 Conn_01x08_Pin, J28 Conn_01x08_Pin, J29 Conn_01x08_Pin, J3 Conn_01x40_Pin, J4 Conn_01x08_Pin, J5 Conn_01x08_Pin, J6 Conn_01x08_Pin, J7 Conn_01x10_Pin, J8 Conn_01x10_Pin, J9 Conn_01x10_Pin, Q1 FDG1024NZ, Q10 FDG1024NZ, Q11 FDG1024NZ, Q12 FDG1024NZ, Q2 FDG1024NZ, Q3 FDG1024NZ, Q4 FDG1024NZ, Q5 FDG1024NZ, Q6 FDG1024NZ, Q7 FDG1024NZ, Q8 FDG1024NZ, Q9 FDG1024NZ, U1 NE555D, U10 74LS161, U11 74LS161, U12 74LS257, U13 74LS257, U14 74LS257, U15 74LS257, U16 74LS245, U17 74LS245, U18 28C256, U19 28C256, U2 74LS161, U20 74LS574, U21 74LS245, U22 74LS245, U23 74LS245, U24 74LS273, U25 74LS574, U26 74LS574, U27 74LS574, U28 HM62256BLP, U29 74LS245, U3 74LS161, U30 74LS245, U31 74LS245, U32 74LS283, U39 74LS283, U4 74LS161, U40 74LS273, U41 74LS273, U42 74LS04, U43 74HC688, U44 74LS574, U45 74LS574, U46 HM62256BLP, U47 74LS574, U48 74LS245, U49 74LS245, U5 74LS161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

Commit message: pushing processor rev1
Piss Quiet reference
Parts:
- added D82: A4, LED_SMD:LED_0603_1608Metric_Pad1.05x0.95mm_HandSolder, symbol Device:LED
- added J30, J35, J40, J42: Conn_01x01_Pin, Connector_PinHeader_2.54mm:PinHeader_1x01_P2.54mm_Vertical, symbol Connector:Conn_01x01_Pin
- added J31, J32, J33, J34, J69: Conn_01x03_Pin, Connector_PinHeader_2.54mm:PinHeader_1x03_P2.54mm_Vertical, symbol Connector:Conn_01x03_Pin
- added J36, J41, J43, J44, J45, J46, J47, J48, J49, J50, J51, J52, J54, J56, J57, J58, J59, J60, J61, J62, J63, J64, J65, J67, J68, J70, J71, J72, J73, J74: J, Connector_PinHeader_2.54mm:PinHeader_1x01_P2.54mm_Vertical, symbol Connector:Conn_01x01_Pin
- added J39: Clock_Aux_Latch_0, Connector_PinHeader_2.54mm:PinHeader_1x01_P2.54mm_Vertical, symbol Connector:Conn_01x01_Pin
- added R141, R142: R, Resistor_SMD:R_0603_1608Metric_Pad0.98x0.95mm_HandSolder, symbol Device:R
- added r140: 470, Resistor_SMD:R_0603_1608Metric_Pad0.98x0.95mm_HandSolder, symbol Device:R
- U1: footprint Package_DIP:DIP-8_W7.62mm_Socket -> Package_SO:SOIC-8_3.9x4.9mm_P1.27mm
Connections:
- net decoder_neg_clock is gone; now on net CLOCK_to_pc_n: U60.5 (E2)
- net decoder_pos_clock is gone; now on net CLOCK_to_pc: U59.6 (E3)
- net reset_n is gone; now on net pc_reset_n: J3.4 (Pin_4)
- net +5V: now also J10.1 (Pin_1), J18.1 (Pin_1), J19.10 (Pin_10), J7.10 (Pin_10), J8.10 (Pin_10), J9.1 (Pin_1), U18.27 (~{WE}), U19.27 (~{WE}), U2.10 (CET), U23.1 (A->B), U29.1 (A->B), U30.1 (A->B), U31.1 (A->B), U40.1 (~{Mr}), U41.1 (~{Mr}), U48.1 (A->B), r139.2, R141.1; no longer U57.6 (E3)
- net 5V_raw: no longer r139.2
- net CLOCK_to_pc: now also U42.5, J32.1 (Pin_1), J32.2 (Pin_2), J32.3 (Pin_3), J33.1 (Pin_1), J33.2 (Pin_2), J33.3 (Pin_3), J34.1 (Pin_1), J34.2 (Pin_2), J34.3 (Pin_3), J67.1 (Pin_1), r140.2
- net GND: now also J11.1 (Pin_1), J12.1 (Pin_1), J12.10 (Pin_10), J13.1 (Pin_1), J13.10 (Pin_10), J18.10 (Pin_10), U18.20 (~{CS}), U18.22 (~{OE}), U19.20 (~{CS}), U19.22 (~{OE}), U44.1 (OE), U45.1 (OE), U47.1 (OE), U49.1 (A->B), U50.1 (A->B), U54.1 (OE), U6.1 (OE), U7.1 (OE), D82.1 (K), R142.1; no longer U58.5 (E2)
- net PC_0: now also J69.1 (Pin_1), J69.2 (Pin_2), J69.3 (Pin_3)
- net clk: now also J1.1 (Pin_1), J2.1 (In)
- net instruction_valid_n: now also J68.1 (Pin_1)
- net pc_reset_n: now also U24.1 (~{Mr})
- net at U55.8: now also J57.1 (Pin_1)
- net at U39.9 (C4): now also J63.1 (Pin_1)
- net at U28.20 (~{CS}): now also J47.1 (Pin_1)
- net at U28.22 (~{OE}): now also J48.1 (Pin_1)
- net at U28.27 (~{WE}): now also J49.1 (Pin_1)
- net at U51.10 (CET): now also U51.7 (CEP), J44.1 (Pin_1)
- net at U51.2 (CP): now also J41.1 (Pin_1)
- net at U51.9 (~{PE}): now also J43.1 (Pin_1)
- net CLOCK_to_pc_n: now reaches U42.6
- net CLOCK_to_pc_n: now also J70.1 (Pin_1)
- net at U49.19 (CE): now also J64.1 (Pin_1)
- net builder_lsb_clock: now reaches J10.10 (Pin_10)
- net builder_lsb_clock: now also U7.11 (Cp)
- net at U45.11 (Cp): now also J45.1 (Pin_1)
- net Data_Bus_OE_n: now reaches U27.1 (OE)
- net Data_Bus_OE_n: now also J11.10 (Pin_10)
- net Data_Bus_Latch_Clock: now reaches U27.11 (Cp)
- net Data_Bus_Latch_Clock: now also J7.1 (Pin_1)
- net at U44.11 (Cp): now also J46.1 (Pin_1)
- net at U32.7 (C0): now also J62.1 (Pin_1)
- net at U29.19 (CE): now also J40.1 (Pin_1)
- net at U25.1 (OE): now also J35.1 (Pin_1)
- net at U25.11 (Cp): now also J8.1 (Pin_1)
- net at J3.6 (Pin_6): now also J31.3 (Pin_3)
- net at J3.7 (Pin_7): now also J31.2 (Pin_2)
- net at J3.8 (Pin_8): now also J31.1 (Pin_1)
- net Load_Constant_OE_n: now reaches J19.9 (Pin_9)
- net Load_Constant_OE_n: now also U31.19 (CE)
- net at U43.1 (G): now also J60.1 (Pin_1)
- net at U40.11 (Cp): now also J54.1 (Pin_1)
- net at U5.15 (TC): now also J42.1 (Pin_1)
- net at U24.11 (Cp): now also J65.1 (Pin_1)
- net at U26.1 (OE): now also J30.1 (Pin_1)
- net at U26.11 (Cp): now also J39.1 (Pin_1)
- net builder_msb_clock: now reaches J9.10 (Pin_10)
- net builder_msb_clock: now also U6.11 (Cp)
- net at U41.11 (Cp): now also J56.1 (Pin_1)
- net at U54.11 (Cp): now also J61.1 (Pin_1)
- net at U50.19 (CE): now also J73.1 (Pin_1)
- net at J21.1: now also J74.1 (Pin_1)
- net at U47.11 (Cp): now also J58.1 (Pin_1)
- net at U23.19 (CE): now also J36.1 (Pin_1)
- net at U21.1 (A->B): now also J71.1 (Pin_1)
- net at U21.19 (CE): now also J72.1 (Pin_1)
- net at U46.20 (~{CS}): now also J50.1 (Pin_1)
- net at U46.22 (~{OE}): now also J51.1 (Pin_1)
- net at U46.27 (~{WE}): now also J52.1 (Pin_1)
- net at U48.19 (CE): now also J59.1 (Pin_1)
- new net: R142.2, U58.5 (E2)
- new net: D82.2 (A), r140.1
- new net: R141.2, U57.6 (E3)
Other:
- note added: "CLOCK"
- note added: "Data Bus Latch"
- note added: "Load Constant Buffer"
- note added: "PC 0 is used to disable the lsb instr buffer and clock the msb instr register"
- note added: "consider using pc_0_n"
