File: processor_attempt_2/processor_attempt_2.kicad_pcb (KiCad board)
At the start: 2 copper layers, 229.9 x 93.3 mm, 275 parts, among them J1 Conn_01x03_Pin, J10 Conn_01x10_Pin, J11 Conn_01x10_Pin, J12 Conn_01x10_Pin, J13 Conn_01x10_Pin, J14 Conn_01x06_Pin, J15 Conn_01x06_Pin, J16 Conn_01x06_Pin, J17 Conn_01x06_Pin, J18 Conn_01x10_Pin, J19 Conn_01x10_Pin, J20 Conn_01x08_Pin, J21 DB9_Female_MountingHoles, J22 Conn_01x08_Pin, J23 Conn_01x08_Pin, J24 Conn_01x08_Pin, J25 Conn_01x08_Pin, J26 Conn_01x08_Pin, J27 Conn_01x08_Pin, J28 Conn_01x08_Pin, J29 Conn_01x08_Pin, J3 Conn_01x40_Pin, J30 J, J31 Conn_01x03_Pin, J32 Conn_01x03_Pin, J33 Conn_01x03_Pin, J34 Conn_01x03_Pin, J36 J, J37 J, J4 Conn_01x08_Pin, J40 Conn_01x01_Pin, J41 J, J42 Conn_01x01_Pin, J43 J, J44 J, J45 J, J46 J, J47 J, J48 J, J49 J, J50 J, J51 J, J52 J, J54 J, J56 J, J57 J, J60 J, J62 J, J63 J, J64 J, J65 J, J67 J, J68 J, J69 Conn_01x03_Pin, J7 Conn_01x10_Pin, J70 J, J73 J, J74 J, J9 Conn_01x10_Pin, U1 NE555D, U18 28C256, U19 28C256, U2 74LS161, U24 74LS273, U27 74LS574, U28 HM62256BLP, U29 74LS245, U3 74LS161, U30 74LS245, U31 74LS245, U32 74LS283, U33 74LS273, U34 74LS273, U35 74LS689, U39 74LS283, U4 74LS161, U40 74LS273, U41 74LS273, U42 74LS04, U46 HM62256BLP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

Commit message: pushing a bunch of new projects
new pcbs
Parts:
- removed G***: LOGO, AudioJacks:star_footprint
- removed G***: LOGO, AudioJacks:plant
- added U56: 74LS04, Package_DIP:DIP-14_W7.62mm_Socket, F.Cu at (33.5, 65.0)
- U1: footprint Package_SO:SOIC-8_3.9x4.9mm_P1.27mm -> Package_DIP:DIP-8_W7.62mm
- moved U33 230.4 mm to (44.5, 89.7), turned to 90 degrees
- moved U34 215.0 mm to (72.4, 89.7), turned to 90 degrees
- moved J32 57.8 mm to (116.0, -3.81)
- moved J33 57.8 mm to (119.0, -3.79)
- moved J34 57.8 mm to (121.9, -3.79)
- moved U57 51.3 mm to (182.1, -14.5)
- moved U58 51.3 mm to (197.4, -14.5)
- moved U59 51.3 mm to (212.6, -14.5)
- moved U60 51.3 mm to (227.8, -14.5)
- moved U28 49.2 mm to (59.7, 107.7)
- moved U46 49.2 mm to (75.6, 100.1)
- moved J11 47.0 mm to (123.3, 76.1)
- moved J19 47.0 mm to (127.1, 76.1)
- moved J18 47.0 mm to (150.0, 63.4)
- moved J7 47.0 mm to (123.2, 63.4)
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Connections:
- net /pc_reset_n renamed /reset_n
- J18 pad 2: /instruction_0 -> /build_constant_0
- J18 pad 3: /instruction_1 -> /build_constant_1
- J18 pad 4: /instruction_2 -> /build_constant_2
- J18 pad 5: /instruction_3 -> /build_constant_3
- J18 pad 6: /instruction_4 -> /build_constant_4
- J18 pad 7: /instruction_5 -> /build_constant_5
- J18 pad 8: /instruction_6 -> /build_constant_6
- J18 pad 9: /instruction_7 -> /build_constant_7
- U31 pad 2: /instruction_0 -> /build_constant_0
- U31 pad 3: /instruction_1 -> /build_constant_1
- U31 pad 4: /instruction_2 -> /build_constant_2
- U31 pad 5: /instruction_3 -> /build_constant_3
- U31 pad 6: /instruction_4 -> /build_constant_4
- U31 pad 7: /instruction_5 -> /build_constant_5
- U31 pad 8: /instruction_6 -> /build_constant_6
- U31 pad 9: /instruction_7 -> /build_constant_7
- U33 pad 12: /mar_4 -> /mar_1
- U33 pad 13: /INTERNAL_BUS_4 -> /INTERNAL_BUS_1
- U33 pad 14: /INTERNAL_BUS_5 -> /INTERNAL_BUS_2
- U33 pad 15: /mar_5 -> /mar_2
- U33 pad 16: /mar_6 -> /mar_5
- U33 pad 17: /INTERNAL_BUS_6 -> /INTERNAL_BUS_5
- U33 pad 18: /INTERNAL_BUS_7 -> /INTERNAL_BUS_6
- U33 pad 19: /mar_7 -> /mar_6
- U33 pad 2: /mar_0 -> /mar_7
- U33 pad 3: /INTERNAL_BUS_0 -> /INTERNAL_BUS_7
- U33 pad 4: /INTERNAL_BUS_1 -> /INTERNAL_BUS_4
- U33 pad 5: /mar_1 -> /mar_4
- U33 pad 6: /mar_2 -> /mar_3
- U33 pad 7: /INTERNAL_BUS_2 -> /INTERNAL_BUS_3
- U33 pad 8: /INTERNAL_BUS_3 -> /INTERNAL_BUS_0
- U33 pad 9: /mar_3 -> /mar_0
Routing:
- net GND: track 1294.4 -> 1093.3 mm
- net +5V: track 1204.5 -> 1040.4 mm, vias 34 -> 33
- net /CLOCK_to_pc: track 246.5 -> 163.4 mm, vias 3 -> 2
- net /instruction_4: track 86.9 -> 24.2 mm, vias 1 -> 0
- net /build_constant_0: track 0.00 -> 41.2 mm
- net /instruction_6: track 98.8 -> 65.1 mm, vias 1 -> 0
- net /instruction_3: track 74.4 -> 42.4 mm, vias 1 -> 0
- net /instruction_7: track 95.8 -> 64.1 mm, vias 1 -> 0
- net /instruction_5: track 88.8 -> 60.3 mm, vias 1 -> 0
- net /reset_n: track 136.2 -> 110.4 mm, vias 5 -> 3
- net /INTERNAL_BUS_7: track 352.4 -> 373.4 mm, vias 8 -> 9
- net /PC_2: track 187.5 -> 169.6 mm
- net /INTERNAL_BUS_3: track 343.2 -> 360.8 mm
- net /instruction_0: track 64.7 -> 47.1 mm, vias 1 -> 0
- net /INTERNAL_BUS_6: track 352.7 -> 369.7 mm, vias 10 -> 11
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Other:
- board text removed: "BOARD CLOCK"
- board text removed: "EXT_CLK"
- board text removed: "ILS_OEn"
- board text removed: "IMS_clk"
- board text removed: "INSTRUCTION LSB"
- board text removed: "INSTRUCTION MSB"
- board text removed: "IVAL_n"
- board text removed: "LOC_CLK"
- board text removed: "PC0"
- board text removed: "SEL_CLK"
