File: processor_attempt_2/processor_attempt_2.kicad_sch (KiCad schematic)
At the start: 297 parts, among them J1 Conn_01x03_Pin, J10 Conn_01x10_Pin, J11 Conn_01x10_Pin, J12 Conn_01x10_Pin, J13 Conn_01x10_Pin, J14 Conn_01x06_Pin, J15 Conn_01x06_Pin, J16 Conn_01x06_Pin, J17 Conn_01x06_Pin, J18 Conn_01x10_Pin, J19 Conn_01x10_Pin, J2 Conn_Coaxial, J20 Conn_01x08_Pin, J21 DB9_Female_MountingHoles, J22 Conn_01x08_Pin, J23 Conn_01x08_Pin, J24 Conn_01x08_Pin, J25 Conn_01x08_Pin, J26 Conn_01x08_Pin, J27 Conn_01x08_Pin, J28 Conn_01x08_Pin, J29 Conn_01x08_Pin, J3 Conn_01x40_Pin, J30 J, J31 Conn_01x03_Pin, J32 Conn_01x03_Pin, J33 Conn_01x03_Pin, J34 Conn_01x03_Pin, J35 Conn_01x01_Pin, J37 J, J39 Clock_Aux_Latch_0, J4 Conn_01x08_Pin, J40 Conn_01x01_Pin, J41 J, J42 Conn_01x01_Pin, J43 J, J44 J, J45 J, J46 J, J47 J, J48 J, J49 J, J5 Conn_01x08_Pin, J50 J, J51 J, J52 J, J54 J, J56 J, J57 J, J6 Conn_01x08_Pin, J60 J, J62 J, J63 J, J64 J, J65 J, J67 J, J68 J, J69 Conn_01x03_Pin, J7 Conn_01x10_Pin, J70 J, J71 J, J72 J, J73 J, J74 J, J8 Conn_01x10_Pin, J9 Conn_01x10_Pin, U1 NE555D, U10 74LS161, U11 74LS161, U12 74LS257, U13 74LS257, U14 74LS257, U15 74LS257, U16 74LS245, U17 74LS245, U18 28C256, U19 28C256, U2 74LS161, U20 74LS574, U21 74LS245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

Commit message: pushing a bunch of new projects
new pcbs
Parts:
- U1: footprint Package_SO:SOIC-8_3.9x4.9mm_P1.27mm -> Package_DIP:DIP-8_W7.62mm
Connections:
- net INTERNAL_BUS_0: now also U33.8 (D3), U34.8 (D3); no longer U33.3 (D0), U34.3 (D0)
- net INTERNAL_BUS_1: now also U33.13 (D4), U34.13 (D4); no longer U33.4 (D1), U34.4 (D1)
- net INTERNAL_BUS_2: now also U33.14 (D5), U34.14 (D5); no longer U33.7 (D2), U34.7 (D2)
- net INTERNAL_BUS_3: now also U33.7 (D2), U34.7 (D2); no longer U33.8 (D3), U34.8 (D3)
- net INTERNAL_BUS_4: now also U33.4 (D1), U34.4 (D1); no longer U33.13 (D4), U34.13 (D4)
- net INTERNAL_BUS_5: now also U33.17 (D6), U34.17 (D6); no longer U33.14 (D5), U34.14 (D5)
- net INTERNAL_BUS_6: now also U33.18 (D7), U34.18 (D7); no longer U33.17 (D6), U34.17 (D6)
- net INTERNAL_BUS_7: now also U33.3 (D0), U34.3 (D0); no longer U33.18 (D7), U34.18 (D7)
- net build_constant_0: now also J18.2 (Pin_2), U31.2 (A0)
- net build_constant_1: now also J18.3 (Pin_3), U31.3 (A1)
- net build_constant_2: now also J18.4 (Pin_4), U31.4 (A2)
- net build_constant_3: now also J18.5 (Pin_5), U31.5 (A3)
- net build_constant_4: now also J18.6 (Pin_6), U31.6 (A4)
- net build_constant_5: now also J18.7 (Pin_7), U31.7 (A5)
- net build_constant_6: now also J18.8 (Pin_8), U31.8 (A6)
- net build_constant_7: now also J18.9 (Pin_9), U31.9 (A7)
- net instruction_0: no longer J18.2 (Pin_2), U31.2 (A0)
- net instruction_1: no longer J18.3 (Pin_3), U31.3 (A1)
- net instruction_2: no longer J18.4 (Pin_4), U31.4 (A2)
- net instruction_3: no longer J18.5 (Pin_5), U31.5 (A3)
- net instruction_4: no longer J18.6 (Pin_6), U31.6 (A4)
- net instruction_5: no longer J18.7 (Pin_7), U31.7 (A5)
- net instruction_6: no longer J18.8 (Pin_8), U31.8 (A6)
- net instruction_7: no longer J18.9 (Pin_9), U31.9 (A7)
- net mar_0: now also U33.9 (Q3); no longer U33.2 (Q0)
- net mar_1: now also U33.12 (Q4); no longer U33.5 (Q1)
- net mar_10: now also U34.15 (Q5); no longer U34.6 (Q2)
- net mar_11: now also U34.6 (Q2); no longer U34.9 (Q3)
- net mar_12: now also U34.5 (Q1); no longer U34.12 (Q4)
- net mar_13: now also U34.16 (Q6); no longer U34.15 (Q5)
- net mar_14: now also U34.19 (Q7); no longer U34.16 (Q6)
- net mar_15: now also U34.2 (Q0); no longer U34.19 (Q7)
- net mar_2: now also U33.15 (Q5); no longer U33.6 (Q2)
- net mar_3: now also U33.6 (Q2); no longer U33.9 (Q3)
- net mar_4: now also U33.5 (Q1); no longer U33.12 (Q4)
- net mar_5: now also U33.16 (Q6); no longer U33.15 (Q5)
- net mar_6: now also U33.19 (Q7); no longer U33.16 (Q6)
- net mar_7: now also U33.2 (Q0); no longer U33.19 (Q7)
- net mar_8: now also U34.9 (Q3); no longer U34.2 (Q0)
- net mar_9: now also U34.12 (Q4); no longer U34.5 (Q1)
- net pc_reset_n renamed reset_n
