File: stepper_motor_controller/stepper_motor_controller_4_for_cnc/stepper_motor_controller_4_for_cnc.kicad_sch (KiCad schematic)
At the start: 45 parts, among them J2 178-009-613R571, U1 74LS74, U11 LM317_TO-220, U3 74LS136

Commit message: mini version
mini
Parts:
- removed R44, R46, R47, R49, R57, R60, R62, R63: 1, Resistor_THT:R_Axial_DIN0204_L3.6mm_D1.6mm_P5.08mm_Horizontal, symbol Device:R
- removed U24, U25, U26, U27: ~, Package_DIP:DIP-8_W7.62mm, symbol my parts:L9110h
