File: stepper_motor_controller/stepper_motor_controller_2/stepper_motor_controller_2.kicad_pcb (KiCad board)
At the start: 2 copper layers, 119.4 x 45.7 mm, 116 parts, among them J2 178-009-613R571, U1 74LS74, U11 LM317_TO-220, U28 74LS74, U3 74LS136

Commit message: sadfj
Parts:
- added D1: LED, LED_SMD:LED_0603_1608Metric, F.Cu at (236.6, 87.1)
- added R91: 1, Resistor_SMD:R_1206_3216Metric, F.Cu at (231.4, 88.6)
Routing:
- net +5V: track 210.8 -> 224.2 mm
- net GND: track 667.1 -> 674.5 mm
- net Net-(D1-K): track 0.00 -> 4.44 mm
