File: stepper_motor_controller/stepper_motor_controller_2/stepper_motor_controller_2.kicad_sch (KiCad schematic)
At the start: 117 parts, among them J2 178-009-613R571, U1 74LS74, U11 LM317_TO-220, U3 74LS136

Commit message: sadfj
Parts:
- added D1: LED, LED_SMD:LED_0603_1608Metric, symbol Device:LED
- added R91: 1, Resistor_SMD:R_1206_3216Metric, symbol Device:R
Connections:
- net +5V: now also D1.2 (A)
- net GND: now also R91.1
- new net: D1.1 (K), R91.2
Changed lines of the file:
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@@
     )
   )
+  (symbol (lib_id "Device:R") (at 302.26 201.93 180) (unit 1)
+    (in_bom yes) (on_board yes) (dnp no) (fields_autoplaced)
+    (property "Reference" "R91" (at 304.8 200.66 0)
+      (effects (font (size 1.27 1.27)) (justify right))
+    )
+    (property "Value" "1" (at 304.8 203.2 0)
+      (effects (font (size 1.27 1.27)) (justify right))
+    )
+    (property "Footprint" "Resistor_SMD:R_1206_3216Metric" (at 304.038 201.93 90)
+      (effects (font (size 1.27 1.27)) hide)
+    )
+    (property "Datasheet" "~" (at 302.26 201.93 0)
+      (effects (font (size 1.27 1.27)) hide)
+    )
+    (pin "1")
+    (pin "2")
+    (instances
+      (project "stepper_motor_controller_2"
+        (path "/4be13624-393a-456f-a51f-7b151a0b69fa"
+          (reference "R91") (unit 1)
+        )
+      )
+    )
+  )
   (symbol (lib_id "Device:R") (at 273.05 43.18 90) (unit 1)
     (in_bom yes) (on_board yes) (dnp no) (fields_autoplaced)
@@
     )
   )
+  (symbol (lib_id "power:GND") (at 302.26 205.74 0) (unit 1)
+    (in_bom yes) (on_board yes) (dnp no) (fields_autoplaced)
+    (property "Reference" "#PWR027" (at 302.26 212.09 0)
+      (effects (font (size 1.27 1.27)) hide)
+    )
+    (property "Value" "GND" (at 302.26 210.82 0)
+      (effects (font (size 1.27 1.27)))
+    )
+    (property "Footprint" "" (at 302.26 205.74 0)
+      (effects (font (size 1.27 1.27)) hide)
+    )
+    (property "Datasheet" "" (at 302.26 205.74 0)
+      (effects (font (size 1.27 1.27)) hide)
+    )
+    (pin "1")
+    (instances
+      (project "stepper_motor_controller_2"
+        (path "/4be13624-393a-456f-a51f-7b151a0b69fa"
+          (reference "#PWR027") (unit 1)
+        )
+      )
+    )
+  )
   (symbol (lib_id "Device:R") (at 347.98 69.85 90) (unit 1)
     (in_bom yes) (on_board yes) (dnp no) (fields_autoplaced)
@@
     )
   )
+  (symbol (lib_id "power:+5V") (at 302.26 190.5 0) (unit 1)
+    (in_bom yes) (on_board yes) (dnp no) (fields_autoplaced)
+    (property "Reference" "#PWR028" (at 302.26 194.31 0)
+      (effects (font (size 1.27 1.27)) hide)
+    )
+    (property "Value" "+5V" (at 302.26 185.42 0)
+      (effects (font (size 1.27 1.27)))
+    )
+    (property "Footprint" "" (at 302.26 190.5 0)
+      (effects (font (size 1.27 1.27)) hide)
+    )
+    (property "Datasheet" "" (at 302.26 190.5 0)
+      (effects (font (size 1.27 1.27)) hide)
+    )
+    (pin "1")
+    (instances
+      (project "stepper_motor_controller_2"
+        (path "/4be13624-393a-456f-a51f-7b151a0b69fa"
+          (reference "#PWR028") (unit 1)
+        )
+      )
+    )
+  )
   (symbol (lib_id "Device:R") (at 271.78 148.59 90) (unit 1)
     (in_bom yes) (on_board yes) (dnp no) (fields_autoplaced)
@@
         )
       )
+    )
+  )
+  (symbol (lib_id "Device:LED") (at 302.26 194.31 90) (unit 1)
+    (in_bom yes) (on_board yes) (dnp no) (fields_autoplaced)
+    (property "Reference" "D1" (at 306.07 194.6275 90)
+      (effects (font (size 1.27 1.27)) (justify right))
+    )
+    (property "Value" "LED" (at 306.07 197.1675 90)
+      (effects (font (size 1.27 1.27)) (justify right))
+    )
+    (property "Footprint" "LED_SMD:LED_0603_1608Metric" (at 302.26 194.31 0)
+      (effects (font (size 1.27 1.27)) hide)
+    )
+    (property "Datasheet" "~" (at 302.26 194.31 0)
+      (effects (font (size 1.27 1.27)) hide)
+    )
+    (pin "1")
+    (pin "2")
+    (instances
+      (project "stepper_motor_controller_2"
+        (path "/4be13624-393a-456f-a51f-7b151a0b69fa"
+          (reference "D1") (unit 1)
+        )
+      )
