File: 93c46a_type/93c46a_type.kicad_pcb (KiCad board)
At the start: 2 copper layers, 132.1 x 83.8 mm, 55 parts, among them J1 Conn_01x40_Pin, J2 Conn_01x03_Pin, U1 93CxxA, U2 74LS123, U3 74LS123, U4 NA555D

Commit message: se
se
Parts:
- removed C2, C3: C, Capacitor_THT:C_Disc_D3.0mm_W2.0mm_P2.50mm
- removed U3: 74LS123, Package_DIP:DIP-16_W7.62mm
- removed r4, r5: 470, Resistor_SMD:R_0603_1608Metric_Pad0.98x0.95mm_HandSolder
- added D2: VCC, LED_SMD:LED_0603_1608Metric_Pad1.05x0.95mm_HandSolder, F.Cu at (54.5, 17.8)
- added D3: VCC, LED_SMD:LED_0603_1608Metric_Pad1.05x0.95mm_HandSolder, F.Cu at (54.5, 20.4)
- added D4: VCC, LED_SMD:LED_0603_1608Metric_Pad1.05x0.95mm_HandSolder, F.Cu at (54.5, 23.0)
- added D5: VCC, LED_SMD:LED_0603_1608Metric_Pad1.05x0.95mm_HandSolder, F.Cu at (54.5, 25.6)
- added J3: Conn_01x03_Pin, Connector_PinHeader_2.54mm:PinHeader_1x03_P2.54mm_Vertical, F.Cu at (53.3, 30.5)
- added JCol1: Conn_01x25_Pin, Connector_PinHeader_2.54mm:PinHeader_1x25_P2.54mm_Vertical, F.Cu at (168.9, 57.1)
- added SW1: SW_SPST, Resistor_THT:R_Axial_DIN0204_L3.6mm_D1.6mm_P5.08mm_Horizontal, F.Cu at (37.6, 34.4)
- added U5: 74LS00, Package_DIP:DIP-14_W7.62mm, F.Cu at (48.3, 76.2)
- added U9: 74HC595, Package_SO:SOIC-16_3.9x9.9mm_P1.27mm, F.Cu at (63.6, 59.1)
- added r10: 470, Resistor_THT:R_Axial_DIN0204_L3.6mm_D1.6mm_P7.62mm_Horizontal, F.Cu at (37.6, 31.3)
- added r11: 470, Resistor_SMD:R_0603_1608Metric_Pad0.98x0.95mm_HandSolder, F.Cu at (48.8, 34.4)
- added r12: 470, Resistor_SMD:R_0603_1608Metric_Pad0.98x0.95mm_HandSolder, F.Cu at (48.8, 36.9)
- added r13: 470, Resistor_SMD:R_0603_1608Metric_Pad0.98x0.95mm_HandSolder, F.Cu at (48.8, 39.5)
- added r8: 470, Resistor_SMD:R_0603_1608Metric_Pad0.98x0.95mm_HandSolder, F.Cu at (48.8, 31.9)
- added r9: 470, Resistor_THT:R_Axial_DIN0204_L3.6mm_D1.6mm_P7.62mm_Horizontal, F.Cu at (37.6, 28.1)
- C5, C6: footprint Capacitor_SMD:C_1206_3216Metric -> Capacitor_THT:C_Disc_D3.0mm_W2.0mm_P2.50mm
- U1: footprint Package_DIP:DIP-8_W7.62mm -> Package_SO:SOIC-8_3.9x4.9mm_P1.27mm
- U4: footprint Package_DIP:DIP-8_W7.62mm_Socket -> Package_DIP:DIP-8_W7.62mm
- r2, r3: footprint Resistor_SMD:R_0603_1608Metric_Pad0.98x0.95mm_HandSolder -> Resistor_THT:R_Axial_DIN0204_L3.6mm_D1.6mm_P7.62mm_Horizontal
- r6, r7: footprint Resistor_SMD:R_1206_3216Metric -> Resistor_THT:R_Axial_DIN0204_L3.6mm_D1.6mm_P7.62mm_Horizontal
- moved C4 67.3 mm to (48.2, 19.3)
- moved C1 60.3 mm to (48.2, 15.7)
- moved C5 46.8 mm to (48.2, 22.8)
- moved C6 46.6 mm to (48.2, 26.4)
- moved r7 45.6 mm to (37.6, 25.0)
- moved r6 45.5 mm to (37.6, 21.8)
- moved r2 45.2 mm to (37.6, 15.5)
- moved r3 44.6 mm to (37.6, 18.7)
- moved D1 41.0 mm to (54.5, 15.2)
- moved U1 40.4 mm to (63.5, 50.8), turned to 180 degrees
- moved r1 28.5 mm to (48.8, 29.4)
- moved U4 15.2 mm to (48.3, 55.9)
Connections:
- U2 pad 10: unconnected-(U2B-B-Pad10) -> /rom_cs
- U2 pad 12: unconnected-(U2B-~{Q}-Pad12) -> /BOOT_read_pulse
- U2 pad 13: unconnected-(U2A-Q-Pad13) -> /rom_cs
- U2 pad 2: unconnected-(U2A-B-Pad2) -> Net-(U2A-B)
- U4 pad 3: unconnected-(U4-Q-Pad3) -> /BOOT_Clock
- U4 pad 4: +5V -> /rom_cs
- r2 pad 1: VCC -> Net-(r10-Pad2)
