File: 93c46a_type/93c46a_type.kicad_sch (KiCad schematic)
At the start: 33 parts, among them J1 Conn_01x40_Pin, J2 Conn_01x03_Pin, U1 93CxxA, U2 74LS123, U3 74LS123, U4 NA555D, U5 74LS00

Commit message: se
se
Parts:
- added D3, D4, D5: VCC, LED_SMD:LED_0603_1608Metric_Pad1.05x0.95mm_HandSolder, symbol Device:LED
- added J3: Conn_01x03_Pin, Connector_PinHeader_2.54mm:PinHeader_1x03_P2.54mm_Vertical, symbol Connector:Conn_01x03_Pin
- added SW1: SW_SPST, Resistor_THT:R_Axial_DIN0204_L3.6mm_D1.6mm_P5.08mm_Horizontal, symbol Switch:SW_SPST
- added U10: 74LS175, symbol 74xx:74LS175
- added U11: 74LS02, symbol 74xx:74LS02
- added U12: 74LS00, symbol 74xx:74LS00
- added U6, U8: 74LS195, symbol 74xx:74LS195
- added U7: 74LS273, symbol 74xx:74LS273
- added U9: 74HC595, Package_SO:SOIC-16_3.9x9.9mm_P1.27mm, symbol 74xx:74HC595
- added r10, r9: 470, Resistor_THT:R_Axial_DIN0204_L3.6mm_D1.6mm_P7.62mm_Horizontal, symbol Device:R
- added r11, r12, r13: 470, Resistor_SMD:R_0603_1608Metric_Pad0.98x0.95mm_HandSolder, symbol Device:R
- C2, C3, J1, J2, JCol1, JCol10, JCol2, JCol3, JCol4, JCol5, JCol6, JCol7, JCol8, JCol9, r4, r5: now not fitted
- C5, C6: footprint Capacitor_SMD:C_1206_3216Metric -> Capacitor_THT:C_Disc_D3.0mm_W2.0mm_P2.50mm; now not fitted
- U1: footprint Package_DIP:DIP-8_W7.62mm -> Package_SO:SOIC-8_3.9x4.9mm_P1.27mm
- U4: footprint Package_DIP:DIP-8_W7.62mm_Socket -> Package_DIP:DIP-8_W7.62mm; now not fitted
- U5: footprint (none) -> Package_DIP:DIP-14_W7.62mm; now not fitted
- r2, r3: footprint Resistor_SMD:R_0603_1608Metric_Pad0.98x0.95mm_HandSolder -> Resistor_THT:R_Axial_DIN0204_L3.6mm_D1.6mm_P7.62mm_Horizontal
- r6, r7: footprint Resistor_SMD:R_1206_3216Metric -> Resistor_THT:R_Axial_DIN0204_L3.6mm_D1.6mm_P7.62mm_Horizontal; now not fitted
Connections:
- net read_pulse is gone; now on net BOOT_read_pulse: U5.1
- net +5V: no longer U4.4 (R)
- net GND: now also U5.14 (VCC), SW1.1 (A), U10.8 (GND), U6.8 (GND), U7.10 (GND), U8.8 (GND), U9.8 (GND), r11.1, r12.1, r13.1
- net VCC: now also U5.7 (GND), U10.16 (VCC), U6.16 (VCC), U7.20 (VCC), U8.16 (VCC), U9.16 (VCC), r10.1, r9.2; no longer r2.1
- net reset_n: now also U10.1 (~{Mr}), U6.1 (~{MR}), U7.1 (~{Mr}), U8.1 (~{MR})
- net rom_cs: now also U2.10 (B), U2.13 (Q), U4.4 (R), D5.2 (A)
- net rom_scl: now also D4.2 (A), J3.2 (Pin_2), U6.10 (CP), U8.10 (CP)
- net rom_sdi: now also D3.2 (A)
- net rom_sdo: now also U8.2 (J), U8.3 (~{K})
- net BOOT_Clock: now reaches U4.3 (Q)
- net BOOT_Clock: now also J3.1 (Pin_1)
- net manual_read: now reaches U5.4
- net manual_read: now also SW1.2 (B), r9.1
- net cpu_request_read_n: now reaches U5.5
- net at U5.6: now also U2.2 (B)
- net BOOT_read_pulse: now reaches U2.12 (~{Q})
- net address_input renamed input_din
- net input_din: now also U6.11 (~{Q3})
- new net: U10.9 (Cp), U11.1
- new net: D3.1 (K), r11.2
- new net: U12.3, U9.12 (RCLK)
- new net: D4.1 (K), r12.2
- new net: D5.1 (K), r13.2
- new net: r10.2, r2.1
- new net input_clock: J3.3 (Pin_3)
- new net instr_reg_0: U7.2 (Q0)
- new net instr_reg_1: U7.5 (Q1)
- new net instr_reg_2: U7.6 (Q2)
- new net instr_reg_3: U7.9 (Q3)
- new net instr_reg_4: U7.12 (Q4)
- new net instr_reg_5: U7.15 (Q5)
- new net instr_reg_6: U7.16 (Q6)
- new net instr_reg_7: U7.19 (Q7)
- new net instruction_parallel_0: U7.3 (D0), U8.15 (Q0)
- new net instruction_parallel_1: U7.4 (D1), U8.14 (Q1)
- new net instruction_parallel_2: U7.7 (D2), U8.13 (Q2)
- new net instruction_parallel_3: U6.2 (J), U6.3 (~{K}), U7.8 (D3), U8.12 (Q3)
- new net instruction_parallel_4: U6.15 (Q0), U7.13 (D4)
- new net instruction_parallel_5: U6.14 (Q1), U7.14 (D5)
- new net instruction_parallel_6: U6.13 (Q2), U7.17 (D6)
- new net instruction_parallel_7: U6.12 (Q3), U7.18 (D7)
- new net parallel_load_instruction_shift_register: U6.9 (~{PE}), U8.9 (~{PE})
Other:
- note added: "555 used to generate BOOT read clock"
- note added: "93C46A SERIAL ROM"
- note added: "INPUT SIGNALS"
- note added: "input din is active low or'd with boot pulse read signal."
- note added: "latch instruction while next instruction is loading"
- note added: "read duration timer. tune to exact # of bytes to read."
- note added: "read pulse generator. must tune to 2cc"
- note added: "request_read_n is low when the cpu requests a read."
- note added: "select from ext clk or boot clk"
- note added: "use nand and invert of two inputs to create or gate"
- moved on the sheet: r2
